File: hardware/kicad/heimdall-switch.kicad_sch (KiCad schematic)
At the start: 42 parts, among them J1 SWD (ARM 10-pin), J2 LOAD_OUT, J3 BATT_IN, J4 B3B-XH-A, Q1 AO3400A, Q2 BSS84, Q3 AO4407A, Q4 AO4407A, Q5 AO3400A, Q6 BSS84, SW1 PTS810, U1 BT832, U2 TPS629206, Y1 32.768kHz

Commit message: J1: generic 2x5 1.27mm header (hanxia C41376037) instead of Samtec
Same ARM 10-pin SMD header at ~$0.10 instead of $1.46. Its recommended
land pattern matches KiCad's PinHeader_2x05_P1.27mm_Vertical_SMD (same
pad width, pitch and row gap; pads 0.1mm shorter at the outer end), so
the footprint and routing stay. Fitted on every board: each needs SWD
once for the bootloader.

Co-Authored-By: Claude Opus 5.5 <noreply@anthropic.com>
Parts:
- J1: LCSC C5155080 -> C41376037
Changed lines of the file:
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@@
 			)
 		)
-		(property "LCSC" "C5155080"
+		(property "LCSC" "C41376037"
 			(at 292.1 111.76 0)
 			(hide yes)

Commit message: Main PCB: SPS-20 style wire entry, board down to 49 x 23 mm
The loop-through relief footprints for J2/J3 took ~14mm of length. Now
plain 0.75mm2 wire pads at the edge and a 2 x 5mm slot between the
battery and load pairs: two tabs, each pair under its own heat shrink.

Everything else shifted 14.5mm left as a block (zones, keep-outs and
locked pre-routes with it). R11 moved to the top side below Q3 so
ADC_FB can reach U1 along the bottom-edge channel; the rest re-routed
with Freerouting plus the usual GND finish/stitch/cleanup steps.
38 vias, ~615mm of track. ERC/DRC clean, full parity.

Co-Authored-By: Claude Opus 5.5 <noreply@anthropic.com>
Parts:
- J2, J3: footprint Connector_Wire:SolderWire-0.75sqmm_1x02_P4.8mm_D1.25mm_OD2.3mm_Relief -> Connector_Wire:SolderWire-0.75sqmm_1x02_P4.8mm_D1.25mm_OD2.3mm
Changed lines of the file:
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@@
 			)
 		)
-		(property "Footprint" "Connector_Wire:SolderWire-0.75sqmm_1x02_P4.8mm_D1.25mm_OD2.3mm_Relief"
+		(property "Footprint" "Connector_Wire:SolderWire-0.75sqmm_1x02_P4.8mm_D1.25mm_OD2.3mm"
 			(at 69.85 102.87 0)
 			(hide yes)
@@
 			)
 		)
-		(property "Footprint" "Connector_Wire:SolderWire-0.75sqmm_1x02_P4.8mm_D1.25mm_OD2.3mm_Relief"
+		(property "Footprint" "Connector_Wire:SolderWire-0.75sqmm_1x02_P4.8mm_D1.25mm_OD2.3mm"
 			(at 160.02 180.34 0)
 			(hide yes)
