File: hardware/kicad-ui/heimdall-switch-ui.kicad_pcb (KiCad board)
At the start: 2 copper layers, 35 x 13 mm, 5 parts, among them J1 B3B-XH-A, SW1 KSC641J

Commit message: UI board GH header, JLC top/bottom export, rev 2 docs with sourced BOM
- UI daughter board: J1 JST-XH B3B-XH-A -> JST-GH BM03B-GHS-TBT
  (vertical SMD, back side, LCSC C161691) to match main board J4;
  re-routed, ERC/DRC clean with parity, renders regenerated.
- jlc_export.py: separate -top/-bottom BOM+CPL sets; bottom angles
  mirrored (180 - angle) as JLC expects, rotation corrections restated
  for that; pad-centre positions; parts without LCSC number left out.
- hardware.md: PCB layout rewritten for rev 2, BOM with board side and
  source links (LCSC/Mouser), UI board and cable BOMs, cost estimate.
- Main board layout pictures and 3D renders regenerated for rev 2.

Co-Authored-By: Claude Opus 5.5 <noreply@anthropic.com>
Parts:
- J1: value B3B-XH-A -> BM03B-GHS-TBT; footprint Connector_JST:JST_XH_B3B-XH-A_1x03_P2.50mm_Vertical -> Connector_JST:JST_GH_BM03B-GHS-TBT_1x03-1MP_P1.25mm_Vertical
- moved J1 2.50 mm to (121.5, 106.0), turned to 90 degrees
Routing:
- net GND: track 24.8 -> 30.0 mm, vias 0 -> 1
- net /LED_A: track 6.50 -> 4.03 mm
- net /BTN: track 20.1 -> 20.7 mm

Commit message: UI board: GH header turned along the board, JLC export for both boards
- UI J1 (BM03B-GHS-TBT) rotated 90 deg and moved left, body >=2mm clear
  of H2's screw hole; runs re-routed, DRC clean with parity.
- UI board plot settings match the main board (Protel extensions, mask
  subtracted from silk, full layer selection: outline and paste were
  being dropped from the Gerbers).
- jlc_export.py takes the project folder as argument
  (python jlc_export.py ../kicad-ui) and zips every Gerber/drill file
  the export writes, whatever the board's layer names.
- hardware.md: board renders and layouts embedded, UI ordering notes.
- gerber/ output folders ignored.

Co-Authored-By: Claude Opus 5.5 <noreply@anthropic.com>
Parts:
- moved J1 0.78 mm to (120.9, 106.5), turned to 0 degrees
Routing:
- net GND: track 30.0 -> 32.1 mm
- net /BTN: track 20.7 -> 19.8 mm

Commit message: UI board: right-angle GH header (same part as main J4)
J1 on the daughter board goes from the vertical BM03B-GHS-TBT to the
right-angle SM03B-GHS-TB, on the back with its opening at the bottom
long edge, so the cable plugs in from the side and both cable ends use
the same header. Re-routed: GND and LED_A to the front through one via
each, BTN on the back to the button's via as before. DRC 0/0 with full
parity, ERC clean; renders and JLC package regenerated.

Order: 15 x SM03B-GHS-TB at TME instead of 10 + 5 x BM03B; TME total
445.6 -> 434.6 SEK. hardware.md updated (UI board, BOM, cost).

Co-Authored-By: Claude Opus 5.5 <noreply@anthropic.com>
Parts:
- J1: value BM03B-GHS-TBT -> SM03B-GHS-TB; footprint Connector_JST:JST_GH_BM03B-GHS-TBT_1x03-1MP_P1.25mm_Vertical -> Connector_JST:JST_GH_SM03B-GHS-TB_1x03-1MP_P1.25mm_Horizontal
- moved J1 3.24 mm to (121.4, 109.7), turned to 180 degrees
Routing:
- net /LED_A: track 4.33 -> 10.4 mm, vias 0 -> 1
- net /BTN: track 19.8 -> 23.6 mm
- net GND: track 32.1 -> 29.3 mm
