File: hardware/kicad-ui/heimdall-switch-ui.kicad_sch (KiCad schematic)
At the start: 3 parts, among them J1 B3B-XH-A, SW1 KSC641J

Commit message: UI daughter board: add two M3 mounting holes
Board grows to 39x13mm with M3 holes 32mm apart at the ends, for a
3D-printed housing on the outside of the hull (LED through the
housing, button sealed with an O-ring). ERC 0/0, DRC clean with
schematic parity.

Co-Authored-By: Claude Opus 5.5 <noreply@anthropic.com>
Parts:
- added H1, H2: M3, MountingHole:MountingHole_3.2mm_M3, symbol Mechanical:MountingHole

Commit message: UI daughter board: tapped M3 holes, board down to 35x13mm
Holes are now 2.5mm M3 tap drill (screws thread into the board from
the housing), so only thread clearance is needed instead of a
head/washer keep-out. Project-local footprint
MountingHole_2.5mm_M3_Tapped. Holes 28.5mm apart. ERC 0/0, DRC clean
with schematic parity.

Co-Authored-By: Claude Opus 5.5 <noreply@anthropic.com>
Parts:
- H1, H2: footprint MountingHole:MountingHole_3.2mm_M3 -> heimdall-switch-ui:MountingHole_2.5mm_M3_Tapped

Commit message: UI board GH header, JLC top/bottom export, rev 2 docs with sourced BOM
- UI daughter board: J1 JST-XH B3B-XH-A -> JST-GH BM03B-GHS-TBT
  (vertical SMD, back side, LCSC C161691) to match main board J4;
  re-routed, ERC/DRC clean with parity, renders regenerated.
- jlc_export.py: separate -top/-bottom BOM+CPL sets; bottom angles
  mirrored (180 - angle) as JLC expects, rotation corrections restated
  for that; pad-centre positions; parts without LCSC number left out.
- hardware.md: PCB layout rewritten for rev 2, BOM with board side and
  source links (LCSC/Mouser), UI board and cable BOMs, cost estimate.
- Main board layout pictures and 3D renders regenerated for rev 2.

Co-Authored-By: Claude Opus 5.5 <noreply@anthropic.com>
Parts:
- J1: value B3B-XH-A -> BM03B-GHS-TBT; footprint Connector_JST:JST_XH_B3B-XH-A_1x03_P2.50mm_Vertical -> Connector_JST:JST_GH_BM03B-GHS-TBT_1x03-1MP_P1.25mm_Vertical; LCSC C144394 -> C161691
Changed lines of the file:
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@@
 			)
 		)
-		(property "Value" "B3B-XH-A"
+		(property "Value" "BM03B-GHS-TBT"
 			(at 101.6 67.31 0)
 			(show_name no)
@@
 			)
 		)
-		(property "Footprint" "Connector_JST:JST_XH_B3B-XH-A_1x03_P2.50mm_Vertical"
+		(property "Footprint" "Connector_JST:JST_GH_BM03B-GHS-TBT_1x03-1MP_P1.25mm_Vertical"
 			(at 101.6 76.2 0)
 			(hide yes)
@@
 			)
 		)
-		(property "LCSC" "C144394"
+		(property "LCSC" "C161691"
 			(at 101.6 76.2 0)
 			(hide yes)

Commit message: Source the prototype run from TME and Mouser
Add hidden Manufacturer/MPN/Supplier/Supplier PN fields to both
schematics for the parts actually ordered; the LCSC fields stay as the
alternative source, so jlc_export.py is unchanged. Mouser takes the
BT832, TPS629206, L1 and Y1, TME the rest.

Substitutes where the original is out of stock or not carried at TME
and Mouser (checked against datasheets and the design notes): Yageo RC
resistors, BSS84AK, CL31A106 (X5R) for C3, Murata 22uF for C4,
DC Components MMSZ5248B, Kingbright L-7104ZGCK LED and Connfly
DS1031-08 SWD header (land pattern within ~0.1mm of the stock
footprint).

order_export.py writes the TME basket import and Mouser BOM files
from the schematic fields; hardware.md's BOM and cost estimate are
updated to the 2026-10-04 prices.

Co-Authored-By: Claude Opus 5.5 <noreply@anthropic.com>
Parts:
- J1: MPN (none) -> BM03B-GHS-TBT(LF)(SN); Manufacturer (none) -> JST; Supplier (none) -> TME; Supplier PN (none) -> BM03B-GHS-TBT
- LED1: MPN (none) -> L-7104ZGCK; Manufacturer (none) -> Kingbright; Supplier (none) -> TME; Supplier PN (none) -> L-7104ZGCK
- SW1: MPN (none) -> KSC641J LFS; Manufacturer (none) -> C&K; Supplier (none) -> TME; Supplier PN (none) -> KSC641JLFS
Changed lines of the file:
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@@
+			)
+		)
+		(property "Manufacturer" "JST"
+			(at 101.6 69.85 0)
+			(hide yes)
+			(show_name no)
+			(do_not_autoplace no)
+			(effects
+				(font
+					(size 1.27 1.27)
+				)
+			)
+		)
+		(property "MPN" "BM03B-GHS-TBT(LF)(SN)"
+			(at 101.6 69.85 0)
+			(hide yes)
+			(show_name no)
+			(do_not_autoplace no)
+			(effects
+				(font
+					(size 1.27 1.27)
+				)
+			)
+		)
+		(property "Supplier" "TME"
+			(at 101.6 69.85 0)
+			(hide yes)
+			(show_name no)
+			(do_not_autoplace no)
+			(effects
+				(font
+					(size 1.27 1.27)
+				)
+			)
+		)
+		(property "Supplier PN" "BM03B-GHS-TBT"
+			(at 101.6 69.85 0)
+			(hide yes)
+			(show_name no)
+			(do_not_autoplace no)
+			(effects
+				(font
+					(size 1.27 1.27)
+				)
 			)
 		)
@@
 			)
 		)
+		(property "Manufacturer" "Kingbright"
+			(at 134.62 76.2 90)
+			(hide yes)
+			(show_name no)
+			(do_not_autoplace no)
+			(effects
+				(font
+					(size 1.27 1.27)
+				)
+			)
+		)
+		(property "MPN" "L-7104ZGCK"
+			(at 134.62 76.2 90)
+			(hide yes)
+			(show_name no)
+			(do_not_autoplace no)
+			(effects
+				(font
+					(size 1.27 1.27)
+				)
+			)
+		)
+		(property "Supplier" "TME"
+			(at 134.62 76.2 90)
+			(hide yes)
+			(show_name no)
+			(do_not_autoplace no)
+			(effects
+				(font
+					(size 1.27 1.27)
+				)
+			)
+		)
+		(property "Supplier PN" "L-7104ZGCK"
+			(at 134.62 76.2 90)
+			(hide yes)
+			(show_name no)
+			(do_not_autoplace no)
+			(effects
+				(font
+					(size 1.27 1.27)
+				)
+			)
+		)
 		(pin "1"
 		)
@@
 			(hide yes)
 			(show_name no)
+			(do_not_autoplace no)
+			(effects
+				(font
+					(size 1.27 1.27)
+				)
+			)
+		)
+		(property "Manufacturer" "C&K"
+			(at 116.84 80.01 90)
+			(hide yes)
+			(show_name no)
+			(do_not_autoplace no)
+			(effects
+				(font
+					(size 1.27 1.27)
+				)
+			)
+		)
+		(property "MPN" "KSC641J LFS"
+			(at 116.84 80.01 90)
+			(hide yes)
+			(show_name no)
+			(do_not_autoplace no)
+			(effects
+				(font
+					(size 1.27 1.27)
+				)
+			)
+		)
+		(property "Supplier" "TME"
+			(at 116.84 80.01 90)
+			(hide yes)
+			(show_name no)
+			(do_not_autoplace no)
+			(effects
+				(font
+					(size 1.27 1.27)
+				)
+			)
+		)
+		(property "Supplier PN" "KSC641JLFS"
+			(at 116.84 80.01 90)
+			(hide yes)
+			(show_name no)

Commit message: UI board: right-angle GH header (same part as main J4)
J1 on the daughter board goes from the vertical BM03B-GHS-TBT to the
right-angle SM03B-GHS-TB, on the back with its opening at the bottom
long edge, so the cable plugs in from the side and both cable ends use
the same header. Re-routed: GND and LED_A to the front through one via
each, BTN on the back to the button's via as before. DRC 0/0 with full
parity, ERC clean; renders and JLC package regenerated.

Order: 15 x SM03B-GHS-TB at TME instead of 10 + 5 x BM03B; TME total
445.6 -> 434.6 SEK. hardware.md updated (UI board, BOM, cost).

Co-Authored-By: Claude Opus 5.5 <noreply@anthropic.com>
Parts:
- J1: value BM03B-GHS-TBT -> SM03B-GHS-TB; footprint Connector_JST:JST_GH_BM03B-GHS-TBT_1x03-1MP_P1.25mm_Vertical -> Connector_JST:JST_GH_SM03B-GHS-TB_1x03-1MP_P1.25mm_Horizontal; LCSC C161691 -> C514175; MPN BM03B-GHS-TBT(LF)(SN) -> SM03B-GHS-TB(LF)(SN); Supplier PN BM03B-GHS-TBT -> SM03B-GHS-TB
Changed lines of the file:
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@@
 			)
 		)
-		(property "Value" "BM03B-GHS-TBT"
+		(property "Value" "SM03B-GHS-TB"
 			(at 101.6 67.31 0)
 			(show_name no)
@@
 			)
 		)
-		(property "Footprint" "Connector_JST:JST_GH_BM03B-GHS-TBT_1x03-1MP_P1.25mm_Vertical"
+		(property "Footprint" "Connector_JST:JST_GH_SM03B-GHS-TB_1x03-1MP_P1.25mm_Horizontal"
 			(at 101.6 76.2 0)
 			(hide yes)
@@
 			)
 		)
-		(property "LCSC" "C161691"
+		(property "LCSC" "C514175"
 			(at 101.6 76.2 0)
 			(hide yes)
@@
 			)
 		)
-		(property "MPN" "BM03B-GHS-TBT(LF)(SN)"
+		(property "MPN" "SM03B-GHS-TB(LF)(SN)"
 			(at 101.6 69.85 0)
 			(hide yes)
@@
 			)
 		)
-		(property "Supplier PN" "BM03B-GHS-TBT"
+		(property "Supplier PN" "SM03B-GHS-TB"
 			(at 101.6 69.85 0)
 			(hide yes)
